File: ki-cad/board/_restore_backup_2026-10-03T17-12-06-818/board.kicad_sch (KiCad schematic)
At the start: 14 parts, among them U1 WEMOS_D1_mini

Commit message: latest ki-cads
Parts:
- F1: footprint Fuse:Fuseholder_Blade_Mini_Keystone_3568 -> Fuse:Fuseholder_Blade_ATO_Littelfuse_Pudenz_2_Pin
Changed lines of the file:
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@@
 			)
 		)
-		(property "Footprint" "Fuse:Fuseholder_Blade_Mini_Keystone_3568"
+		(property "Footprint" "Fuse:Fuseholder_Blade_ATO_Littelfuse_Pudenz_2_Pin"
 			(at 120.65 62.738 90)
 			(hide yes)
